File: KiCAD/KZ80-MSXMEM.kicad_pcb (KiCad board)
At the start: 2 copper layers, 100 x 75 mm, 13 parts, among them J1 SBC8080 BUS, J2 MSX SLOT, U1 74HC00, U2 SRAM128kbit, U3 28C256

Commit message: REV2 64kB Version ガーバー出力
Parts:
- added JP1: RAM SIZE, Jumper:SolderJumper-3_P1.3mm_Bridged12_RoundedPad1.0x1.5mm, F.Cu at (229.2, 76.4)
- added R1: 10k, Resistor_THT:R_Axial_DIN0207_L6.3mm_D2.5mm_P10.16mm_Horizontal, F.Cu at (229.1, 91.2)
- U2: value SRAM128kbit -> 628128; footprint Package_DIP:DIP-28_W15.24mm_Socket_LongPads -> Package_DIP:DIP-32_W15.24mm_Socket_LongPads
- moved U2 0.96 mm to (209.0, 76.6)
Connections:
- J1 pad 17: (no net) -> unconnected-(J1-Pad17)
- J1 pad 18: /~MEMR -> /~{MEMR}
- J1 pad 19: (no net) -> unconnected-(J1-Pad19)
- J1 pad 20: /~MEMW -> /~{MEMW}
- J1 pad 21: (no net) -> unconnected-(J1-Pad21)
- J1 pad 22: (no net) -> unconnected-(J1-Pad22)
- J1 pad 23: (no net) -> unconnected-(J1-Pad23)
- J1 pad 24: (no net) -> unconnected-(J1-Pad24)
- J1 pad 5: (no net) -> unconnected-(J1-Pad5)
- J1 pad 6: (no net) -> unconnected-(J1-Pad6)
- J1 pad 7: (no net) -> unconnected-(J1-Pad7)
- J1 pad 8: (no net) -> unconnected-(J1-Pad8)
- J2 pad 2: (no net) -> unconnected-(J2-Pad2)
- J2 pad 3: (no net) -> unconnected-(J2-Pad3)
- J2 pad 5: (no net) -> unconnected-(J2-Pad5)
- U1 pad 11: Net-(U1-Pad11) -> /~{SRAMCS}
- U1 pad 12: /A15 -> Net-(JP1-Pad2)
- U2 pad 1: /A14 -> unconnected-(U2-Pad1)
- U2 pad 10: /A0 -> /A2
- U2 pad 11: /D0 -> /A1
- U2 pad 12: /D1 -> /A0
- U2 pad 13: /D2 -> /D0
- U2 pad 14: GND -> /D1
- U2 pad 15: /D3 -> /D2
- U2 pad 16: /D4 -> GND
- U2 pad 17: /D5 -> /D3
- U2 pad 18: /D6 -> /D4
- U2 pad 19: /D7 -> /D5
- U2 pad 2: /A12 -> GND
- U2 pad 20: Net-(U1-Pad11) -> /D6
- U2 pad 21: /A10 -> /D7
- U2 pad 22: /~MEMR -> /~{SRAMCS}
- U2 pad 23: /A11 -> /A10
- U2 pad 24: /A9 -> /~{MEMR}
- U2 pad 25: /A8 -> /A11
- U2 pad 26: /A13 -> /A9
- U2 pad 27: /~MEMW -> /A8
- U2 pad 28: VCC -> /A13
- U2 pad 3: /A7 -> /A14
- U2 pad 4: /A6 -> /A12
- U2 pad 5: /A5 -> /A7
- U2 pad 6: /A4 -> /A6
- U2 pad 7: /A3 -> /A5
- U2 pad 8: /A2 -> /A4
- U2 pad 9: /A1 -> /A3
- U3 pad 22: /~MEMR -> /~{MEMR}
Routing:
- net /~{MEMR}: track 0.00 -> 72.4 mm
- net /~{SRAMCS}: track 0.00 -> 70.5 mm
- net Net-(U1-Pad11): track 63.8 -> 0.00 mm, vias 1 -> 0
- net Net-(JP1-Pad2): track 0.00 -> 63.2 mm
- net /~MEMR: track 57.9 -> 0.00 mm
- net /~{MEMW}: track 0.00 -> 46.8 mm
- net /~MEMW: track 42.7 -> 0.00 mm
- net /A13: track 47.6 -> 75.2 mm
- net /A15: track 72.1 -> 93.8 mm
- net VCC: track 83.6 -> 104.2 mm
- net Net-(J2-Pad4): track 94.3 -> 109.4 mm
- net /A11: track 62.2 -> 76.2 mm
- net Net-(J2-Pad1): track 97.5 -> 107.5 mm
- net /A0: track 59.4 -> 69.3 mm, vias 1 -> 0
- net /A8: track 48.2 -> 57.2 mm
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Other:
- net class BOLD removed
- net class Default removed
- board text added: "SRAM"
- board text added: "[KZ80-MSXMEM] MSX Memory Board REV2 64kB Version / KUNI-NET 2022"
- board text added: "~{SLT0}"
- board text added: "~{SLT2}"
- board text added: "~{SLT3}"
- board text removed: "128k(32kB) SRAM"
- board text removed: "[KZ80-MSXMEM] MSX Memory Board REV1 KUNI-NET 2021"
- board text removed: "~SLT0"
- board text removed: "~SLT2"
- board text removed: "~SLT3"
